File: ElectricalDiagram.kicad_sch (KiCad schematic)
At the start: 29 parts

Commit message: updated schems to KiCAD V10, updated submodules to point to current version
Parts:
- U1, U10, U11, U12, U13, U14, U15, U16, U17, U18, U19, U2, U20, U21, U22, U23, U24, U25, U26, U27, U28, U29, U3, U4, U5, U6, U7, U8, U9: value ~ -> (none)
Connections:
- net at U27. (CANL): no longer U28. (GND)
- net at U3. (Ref_Out): now also U4. (Ref_Out)
- net at U4. (Ref_Out): no longer U3. (Ref_Out)
- new net: U10. (7-Pin), U12. (7-Pin) (x3)
- new net: U5. (7-Pin), U7. (7-Pin) (x3)
- new net: U11. (7-Pin), U13. (7-Pin) (x3)
- new net: U14. (7-Pin), U15. (7-Pin) (x3)
- new net: U24. (7-Pin), U25. (7-Pin) (x3)
- new net: U27. (CANL), U28. (GND)
- new net: U8. (7-Pin), U9. (7-Pin) (x3)
- new net: U22. (7-Pin), U23. (7-Pin) (x3)
- new net: U20. (7-Pin), U21. (7-Pin) (x3)
- new net: U16. (7-Pin), U17. (7-Pin) (x3)
- new net: U18. (7-Pin), U19. (7-Pin) (x3)
